Commit message: change model

File: description/camera.xacro (robot description, xacro)
@@ -4,5 +4,5 @@
     <xacro:property name="camera_width"              value="0.03"/>
     <xacro:property name="camera_height"             value="0.03"/>
-    <xacro:property name="camera_offset_x"           value="0.318"/>
+    <xacro:property name="camera_offset_x"           value="0.210"/>
     <xacro:property name="camera_offset_z"           value="0.063"/>
     <!-- Camera -->

File: description/depth_camera.xacro (robot description, xacro)
@@ -4,5 +4,5 @@
     <xacro:property name="RGBD_width"              value="0.09"/>
     <xacro:property name="RGBD_height"             value="0.03"/>
-    <xacro:property name="RGBD_offset_x"           value="0.318"/>
+    <xacro:property name="RGBD_offset_x"           value="0.210"/>
     <xacro:property name="RGBD_offset_z"           value="0.063"/>
     <!-- RGB_Depth camera -->

File: description/gz_diff_drive_control.xacro (robot description, xacro)
@@ -7,6 +7,6 @@
             <left_joint>left_wheel_joint</left_joint>
             <right_joint>right_wheel_joint</right_joint>
-            <wheel_separation>0.266</wheel_separation>
-            <wheel_radius>0.034</wheel_radius>
+            <wheel_separation>0.060</wheel_separation>
+            <wheel_radius>0.035</wheel_radius>
             <!-- Limits -->
             <max_wheel_torque>200</max_wheel_torque>

File: description/lidar.xacro (robot description, xacro)
@@ -3,5 +3,5 @@
     <xacro:property name="lidar_radius"             value="0.025"/>
     <xacro:property name="lidar_thickness"          value="0.040"/>
-    <xacro:property name="lidar_offset_x"           value="0.230"/>
+    <xacro:property name="lidar_offset_x"           value="0.105"/>
     <xacro:property name="lidar_offset_z"           value="0.098"/>
     <!-- Lidar -->

File: description/robot_main.xacro (robot description, xacro)
@@ -2,17 +2,17 @@
 <robot xmlns:xacro="http://www.ros.org/wiki/xacro">
     <xacro:include filename = "inertial_macros.xacro" />
-    <xacro:property name="chassis_length"           value="0.320"/>
-    <xacro:property name="chassis_width"            value="0.240"/>
-    <xacro:property name="chassis_height"           value="0.078"/>
+    <xacro:property name="chassis_length"           value="0.210"/>
+    <xacro:property name="chassis_width"            value="0.103"/>
+    <xacro:property name="chassis_height"           value="0.090"/>
     <xacro:property name="chassis_mass"             value="0.700"/>
-    <xacro:property name="wheel_radius"             value="0.034"/>
-    <xacro:property name="wheel_thickness"          value="0.026"/>
+    <xacro:property name="wheel_radius"             value="0.035"/>
+    <xacro:property name="wheel_thickness"          value="0.025"/>
     <xacro:property name="wheel_mass"               value="0.050"/>
-    <xacro:property name="wheel_offset_x"           value="0.133"/>
-    <xacro:property name="wheel_offset_y"           value="0.133"/>
+    <xacro:property name="wheel_offset_x"           value="0.085"/>
+    <xacro:property name="wheel_offset_y"           value="0.033"/>
     <xacro:property name="wheel_offset_z"           value="0.020"/>
     <xacro:property name="caster_wheel_radius"      value="${wheel_radius - wheel_offset_z}"/>
     <xacro:property name="caster_wheel_mass"        value="0.010"/>
-    <xacro:property name="caster_wheel_offset_x"    value="0.230"/>
+    <xacro:property name="caster_wheel_offset_x"    value="0.200"/>
     <xacro:property name="caster_wheel_offset_z"    value="${wheel_offset_z - wheel_radius + caster_wheel_radius}"/>
     <!-- Colors -->

File: description/ros2_control.xacro (robot description, xacro)
@@ -8,6 +8,6 @@
                     <param name="right_wheel_name">right_wheel_joint</param>
                     <param name="loop_rate">30</param>
-                    <param name="device">/dev/ttyUSB1</param>
-                    <param name="baud_rate">115200</param>
+                    <param name="device">/dev/ttyUSB3</param>
+                    <param name="baud_rate">256000</param>
                     <param name="timeout_ms">1000</param>
                     <param name="enc_counts_per_rev">616</param>
